File: hackpad/hackpad.kicad_sch (KiCad schematic)
At the start: 0 parts

Commit message: update (06/11/2025)
-finished schematic
-finished pcb design
Parts:
- added D1, D2, D3, D4: SK6812MINI, LED_SMD:LED_SK6812MINI_PLCC4_3.5x3.5mm_P1.75mm, symbol LED:SK6812MINI
- added SW1, SW2, SW3, SW4: SW_Push, Button_Switch_Keyboard:SW_Cherry_MX_1.00u_PCB, symbol Switch:SW_Push
- added U1: XIAO-RP2040-DIP, OPL:XIAO-RP2040-DIP, symbol OPL:XIAO-RP2040-DIP
- added U3: ~, OLED:SSD1306-0.91-OLED-4pin-128x32, symbol OLED:_1
Connections:
- new net: SW4.2, U1.10 (GPIO4/MISO)
- new net: D3.1 (DOUT), D4.3 (DIN)
- new net: D1.3 (DIN), D2.1 (DOUT)
- new net: D2.3 (DIN), U1.11 (GPIO3/MOSI)
- new net: SW3.2, U1.9 (GPIO2/SCK)
- new net: SW1.2, U1.7 (GPIO0/TX)
- new net: D1.1 (DOUT), D3.3 (DIN)
- new net: U1.5 (GPIO6/SDA), U3.4 (SDA)
- new net: U1.6 (GPIO7/SCL), U3.3 (SCL)
- new net: SW2.2, U1.8 (GPIO1/RX)
- new net +5V: D1.4 (VDD), D2.4 (VDD), D3.4 (VDD), D4.4 (VDD), U1.14 (VBUS), U3.2 (VCC)
- new net GND: D1.2 (VSS), D2.2 (VSS), D3.2 (VSS), D4.2 (VSS), SW1.1, SW2.1, SW3.1, SW4.1, U1.13 (GND), U3.1 (GND)
Other:
- note added: "OLED"
